Commit message: update robot model

File: robot_p/model/robot-p.urdf.xacro (robot description, xacro)
@@ -2,4 +2,9 @@
 <robot xmlns:xacro="http://ros.org/wiki/xacro"  name="robot-p">
   <link name="base_link">
+    <inertial>
+      <origin rpy="0 0 0" xyz="0.0 0.0 0.0"/>
+      <mass value="0.56"/>
+      <inertia ixx="0.004878" ixy="-6.2341e-07" ixz="-7.4538e-07" iyy="0.00090164" iyz="-0.00014394" izz="0.0042946"/>
+    </inertial>
     <visual>
       <geometry>
@@ -11,6 +16,12 @@
     </visual>
   </link>
-  <xacro:include filename="$(find robot_p)/model/robot-p_rear_wheel.urdf.xacro" />
-  <xacro:include filename="$(find robot_p)/model/robot-p_front_wheel.urdf.xacro" />
-  <xacro:include filename="$(find robot_p)/model/robot-p_laser_scanner.urdf.xacro" />
+  <collision>
+  	<geometry>
+  		<box size="0.39 0.45 0.12"/>
+  	</geometry>
+  </collision>
+  <xacro:include filename="$(find robot_p_model)/urdf/robot-p_rear_wheel.urdf.xacro" />
+  <xacro:include filename="$(find robot_p_model)/urdf/robot-p.gazebo" />
+  <xacro:include filename="$(find robot_p_model)/urdf/robot-p_front_wheel.urdf.xacro" />
+  <xacro:include filename="$(find robot_p_model)/urdf/robot-p_laser_scanner.urdf.xacro" />
 </robot>

File: robot_p/model/robot-p_front_wheel.urdf.xacro (robot description, xacro)
@@ -2,4 +2,9 @@
 <robot xmlns:xacro="http://ros.org/wiki/xacro">
   <link name="front_left_wheel">
+    <inertial>
+      <origin rpy="0 0 0" xyz="0.0 0.0 0.0"/>
+      <mass value="0.56"/>
+      <inertia ixx="0.004878" ixy="-6.2341e-07" ixz="-7.4538e-07" iyy="0.00090164" iyz="-0.00014394" izz="0.0042946"/>
+    </inertial>
     <visual>
       <geometry>
@@ -11,11 +16,23 @@
       <origin xyz="0 0 0" rpy="${-3.1415927/2.0} 0 0" />
     </visual>
+    <collision>
+      <origin xyz="0 0 0" rpy="${-3.1415927/2.0} 0 0" />
+      <geometry>
+        <cylinder length="0.05" radius="0.105"/>
+      </geometry>
+    </collision>
   </link>
-  <joint name="base_to_front_left_wheel" type="fixed">
+  <joint name="base_to_front_left_wheel" type="continuous">
     <origin xyz="0.07 0.175 -0.075"/>
+    <axis xyz="0 1 0" />
     <parent link="base_link"/>
     <child link="front_left_wheel"/>
   </joint>
   <link name="front_right_wheel">
+    <inertial>
+      <origin rpy="0 0 0" xyz="0.0 0.0 0.0"/>
+      <mass value="0.56"/>
+      <inertia ixx="0.004878" ixy="-6.2341e-07" ixz="-7.4538e-07" iyy="0.00090164" iyz="-0.00014394" izz="0.0042946"/>
+    </inertial>
     <visual>
       <geometry>
@@ -27,6 +44,13 @@
       <origin xyz="0 0 0" rpy="${-3.1415927/2.0} 0 0" />
     </visual>
+    <collision>
+      <origin xyz="0 0 0" rpy="${-3.1415927/2.0} 0 0" />
+      <geometry>
+        <cylinder length="0.05" radius="0.105"/>
+      </geometry>
+    </collision>
   </link>
-  <joint name="base_to_right_left_wheel" type="fixed">
+  <joint name="base_to_right_left_wheel" type="continuous">
+    <axis xyz="0 -1 0" />
     <origin xyz="0.07 -0.175 -0.075"/>
     <parent link="base_link"/>

File: robot_p/model/robot-p_laser_scanner.urdf.xacro (robot description, xacro)
@@ -2,4 +2,9 @@
 <robot xmlns:xacro="http://ros.org/wiki/xacro">
   <link name="laser_scanner">
+    <inertial>
+      <origin rpy="0 0 0" xyz="0.0 0.0 0.0"/>
+      <mass value="0.56"/>
+      <inertia ixx="0.004878" ixy="-6.2341e-07" ixz="-7.4538e-07" iyy="0.00090164" iyz="-0.00014394" izz="0.0042946"/>
+    </inertial>
     <visual>
       <geometry>
@@ -11,4 +16,9 @@
       <origin xyz="0 0 0"/>
     </visual>
+    <collision>
+      <geometry>
+        <box size="0.1 .07 .06"/>
+      </geometry>
+    </collision>
   </link>
   <joint name="laser_pillar_to_laser_scanner" type="fixed">
@@ -18,4 +28,9 @@
   </joint>
   <link name="laser_pillar">
+    <inertial>
+      <origin rpy="0 0 0" xyz="0.0 0.0 0.0"/>
+      <mass value="0.56"/>
+      <inertia ixx="0.004878" ixy="-6.2341e-07" ixz="-7.4538e-07" iyy="0.00090164" iyz="-0.00014394" izz="0.0042946"/>
+    </inertial>
     <visual>
       <geometry>
@@ -27,4 +42,9 @@
       <origin xyz="0 0 0"/>
     </visual>
+    <collision>
+      <geometry>
+        <box size="0.1 .07 .06"/>
+      </geometry>
+    </collision>
   </link>
   <joint name="base_to_laser_pillar" type="fixed">

File: robot_p/model/robot-p_rear_wheel.urdf.xacro (robot description, xacro)
@@ -2,4 +2,9 @@
 <robot xmlns:xacro="http://ros.org/wiki/xacro">
   <link name="rear_left_swivel">
+    <inertial>
+      <origin rpy="0 0 0" xyz="0.0 0.0 0.0"/>
+      <mass value="0.56"/>
+      <inertia ixx="0.004878" ixy="-6.2341e-07" ixz="-7.4538e-07" iyy="0.00090164" iyz="-0.00014394" izz="0.0042946"/>
+    </inertial>
     <visual>
       <origin xyz="0 0 0" rpy="0 0 0"/>
@@ -11,7 +16,13 @@
       </material>
     </visual>
+    <collision>
+      <geometry>
+        <box size="0.06 0.026 0.075"/>
+      </geometry>
+    </collision>
   </link>
-  <joint name="base_rear_left_swivel_joint" type="fixed">
+  <joint name="base_rear_left_swivel_joint" type="continuous">
     <origin xyz="-0.155 0.185 -0.0975" rpy="0 0 0"/>
+    <axis xyz="0 0 1" />
     <anchor xyz="0 1 0"/>
     <limit effort="100" velocity="100" k_velocity="0" />
@@ -21,4 +32,9 @@
   </joint>
   <link name="rear_left_center_wheel">
+    <inertial>
+      <origin rpy="0 0 0" xyz="0.0 0.0 0.0"/>
+      <mass value="0.56"/>
+      <inertia ixx="0.004878" ixy="-6.2341e-07" ixz="-7.4538e-07" iyy="0.00090164" iyz="-0.00014394" izz="0.0042946"/>
+    </inertial>
     <visual>
       <origin xyz="0 0 0" rpy="${-3.1415927/2.0} 0 0"/>
@@ -30,6 +46,12 @@
       </material>
     </visual>
+    <collision>
+      <origin xyz="0 0 0" rpy="${-3.1415927/2.0} 0 0"/>
+      <geometry>
+        <cylinder length="0.025" radius="0.05"/>
+      </geometry>
+    </collision>
   </link>
-  <joint name="rear_left_swivel_wheel_joint" type="fixed">
+  <joint name="rear_left_swivel_wheel_joint" type="continuous">
     <origin xyz="-0.03 0 -0.0375" rpy="0 0 0"/>
     <axis xyz="0 1 0"/>
@@ -41,4 +63,9 @@
   </joint>
   <link name="rear_right_swivel">
+    <inertial>
+      <origin rpy="0 0 0" xyz="0.0 0.0 0.0"/>
+      <mass value="0.56"/>
+      <inertia ixx="0.004878" ixy="-6.2341e-07" ixz="-7.4538e-07" iyy="0.00090164" iyz="-0.00014394" izz="0.0042946"/>
+    </inertial>
     <visual>
       <origin xyz="0 0 0" rpy="0 0 0"/>
@@ -50,7 +77,13 @@
       </material>
     </visual>
+    <collision>
+      <geometry>
+        <box size="0.06 0.026 0.075"/>
+      </geometry>
+    </collision>
   </link>
-  <joint name="base_rear_right_swivel_joint" type="fixed">
+  <joint name="base_rear_right_swivel_joint" type="continuous">
     <origin xyz="-0.155 -0.185 -0.0975" rpy="0 0 0"/>
+    <axis xyz="0 0 1" />
     <anchor xyz="0 1 0"/>
     <limit effort="100" velocity="100" k_velocity="0" />
@@ -60,4 +93,9 @@
   </joint>
   <link name="rear_right_center_wheel">
+    <inertial>
+      <origin rpy="0 0 0" xyz="0.0 0.0 0.0"/>
+      <mass value="0.56"/>
+      <inertia ixx="0.004878" ixy="-6.2341e-07" ixz="-7.4538e-07" iyy="0.00090164" iyz="-0.00014394" izz="0.0042946"/>
+    </inertial>
     <visual>
       <origin xyz="0 0 0" rpy="${-3.1415927/2.0} 0 0"/>
@@ -69,6 +107,12 @@
       </material>
     </visual>
+    <collision>
+      <origin xyz="0 0 0" rpy="${-3.1415927/2.0} 0 0"/>
+      <geometry>
+        <cylinder length="0.025" radius="0.05"/>
+      </geometry>
+    </collision>
   </link>
-  <joint name="rear_right_swivel_wheel_joint" type="fixed">
+  <joint name="rear_right_swivel_wheel_joint" type="continuous">
     <origin xyz="-0.03 0 -0.0375" rpy="0 0 0"/>
     <axis xyz="0 1 0"/>
