Commit message: Fixes URDF files + rotation

File: robot_p/model/robot-p_front_wheel.urdf.xacro (robot description, xacro)
@@ -23,5 +23,5 @@
     </collision>
   </link>
-  <joint name="base_to_front_left_wheel" type="continuous">
+  <joint name="base_to_front_left_wheel" type="fixed">
     <origin xyz="0.07 0.175 -0.075"/>
     <axis xyz="0 1 0" />
@@ -51,5 +51,5 @@
     </collision>
   </link>
-  <joint name="base_to_right_left_wheel" type="continuous">
+  <joint name="base_to_right_left_wheel" type="fixed">
     <axis xyz="0 -1 0" />
     <origin xyz="0.07 -0.175 -0.075"/>

File: robot_p/model/robot-p_laser_scanner.urdf.xacro (robot description, xacro)
@@ -23,5 +23,5 @@
   </link>
   <joint name="laser_pillar_to_laser_scanner" type="fixed">
-    <origin xyz="0.0 0 0.06"/>
+    <origin xyz="0.0 0 0.06" rpy="0.0 0.0 3.1416"/>
     <parent link="laser_pillar"/>
     <child link="laser_scanner"/>

File: robot_p/model/robot-p_rear_wheel.urdf.xacro (robot description, xacro)
@@ -22,5 +22,5 @@
     </collision>
   </link>
-  <joint name="base_rear_left_swivel_joint" type="continuous">
+  <joint name="base_rear_left_swivel_joint" type="fixed">
     <origin xyz="-0.155 0.185 -0.0975" rpy="0 0 0"/>
     <axis xyz="0 0 1" />
@@ -53,5 +53,5 @@
     </collision>
   </link>
-  <joint name="rear_left_swivel_wheel_joint" type="continuous">
+  <joint name="rear_left_swivel_wheel_joint" type="fixed">
     <origin xyz="-0.03 0 -0.0375" rpy="0 0 0"/>
     <axis xyz="0 1 0"/>
@@ -83,5 +83,5 @@
     </collision>
   </link>
-  <joint name="base_rear_right_swivel_joint" type="continuous">
+  <joint name="base_rear_right_swivel_joint" type="fixed">
     <origin xyz="-0.155 -0.185 -0.0975" rpy="0 0 0"/>
     <axis xyz="0 0 1" />
@@ -114,5 +114,5 @@
     </collision>
   </link>
-  <joint name="rear_right_swivel_wheel_joint" type="continuous">
+  <joint name="rear_right_swivel_wheel_joint" type="fixed">
     <origin xyz="-0.03 0 -0.0375" rpy="0 0 0"/>
     <axis xyz="0 1 0"/>
